File: PCB/ZXTeensyIF1.kicad_sch (KiCad schematic)
At the start: 15 parts, among them Q10 ZTX313, Q11 ZTX313, U1 LA15-302, U4 74HC04, X1 8Mhz

Commit message: feat: Upload initial PCB v0.3
Parts:
- C3, C4: footprint Resistor_THT:R_Axial_DIN0207_L6.3mm_D2.5mm_P10.16mm_Horizontal -> Capacitor_THT:C_Disc_D3.4mm_W2.1mm_P2.50mm
- R35: footprint Resistor_THT:R_Axial_DIN0207_L6.3mm_D2.5mm_P10.16mm_Horizontal -> Resistor_THT:R_Axial_DIN0207_L6.3mm_D2.5mm_P7.62mm_Horizontal
Other:
- title: ZXTeensyIF1 -> ${PRJ_NAME}
- moved on the sheet: C5, C6, U4G
Changed lines of the file:
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@@
 	(paper "A4")
 	(title_block
-		(title "ZXTeensyIF1")
-		(date "2026-01-04")
-		(rev "0.1")
+		(title "${PRJ_NAME}")
+		(date "${PRJ_DATE}")
+		(rev "${PRJ_REVISION}")
+	)
+	(junction
+		(at 123.19 26.67)
+		(diameter 0)
+		(color 0 0 0 0)
 	)
 	(junction
@@
 	)
 	(junction
-		(at 166.37 19.05)
+		(at 166.37 26.67)
 		(diameter 0)
 		(color 0 0 0 0)
@@
 	)
 	(junction
-		(at 185.42 31.75)
+		(at 185.42 39.37)
 		(diameter 0)
 		(color 0 0 0 0)
@@
 	)
 	(junction
-		(at 166.37 31.75)
+		(at 166.37 39.37)
 		(diameter 0)
 		(color 0 0 0 0)
@@
 	)
 	(junction
-		(at 123.19 19.05)
-		(diameter 0)
-		(color 0 0 0 0)
-	)
-	(junction
 		(at 88.9 54.61)
 		(diameter 0)
@@
 	)
 	(junction
-		(at 147.32 19.05)
+		(at 147.32 26.67)
 		(diameter 0)
 		(color 0 0 0 0)
@@
 	(wire
 		(pts
-			(xy 166.37 29.21) (xy 166.37 31.75)
+			(xy 166.37 36.83) (xy 166.37 39.37)
 		)
 		(stroke
@@
 	(wire
 		(pts
-			(xy 177.8 24.13) (xy 181.61 24.13)
-		)
-		(stroke
-			(width 0)
-			(type default)
-		)
-	)
-	(wire
-		(pts
-			(xy 147.32 31.75) (xy 147.32 29.21)
+			(xy 147.32 39.37) (xy 147.32 36.83)
 		)
 		(stroke
@@
 	(wire
 		(pts
-			(xy 123.19 19.05) (xy 123.19 30.48)
+			(xy 140.97 88.9) (xy 133.35 88.9)
 		)
 		(stroke
@@
 	(wire
 		(pts
-			(xy 140.97 88.9) (xy 133.35 88.9)
+			(xy 88.9 57.15) (xy 88.9 59.69)
 		)
 		(stroke
@@
 	(wire
 		(pts
-			(xy 88.9 57.15) (xy 88.9 59.69)
+			(xy 88.9 49.53) (xy 88.9 52.07)
 		)
 		(stroke
@@
 	(wire
 		(pts
-			(xy 88.9 49.53) (xy 88.9 52.07)
+			(xy 166.37 26.67) (xy 166.37 29.21)
 		)
 		(stroke
@@
 	(wire
 		(pts
-			(xy 166.37 19.05) (xy 166.37 21.59)
+			(xy 123.19 16.51) (xy 123.19 26.67)
 		)
 		(stroke
@@
 	(wire
 		(pts
-			(xy 185.42 31.75) (xy 166.37 31.75)
+			(xy 185.42 39.37) (xy 166.37 39.37)
 		)
 		(stroke
@@
 	(wire
 		(pts
-			(xy 185.42 31.75) (xy 208.28 31.75)
+			(xy 185.42 39.37) (xy 208.28 39.37)
 		)
 		(stroke
@@
 	(wire
 		(pts
-			(xy 177.8 24.13) (xy 177.8 19.05)
-		)
-		(stroke
-			(width 0)
-			(type default)
-		)
-	)
-	(wire
-		(pts
 			(xy 102.87 185.42) (xy 106.68 185.42)
 		)
@@
 	(wire
 		(pts
-			(xy 147.32 19.05) (xy 147.32 21.59)
+			(xy 147.32 26.67) (xy 147.32 29.21)
 		)
 		(stroke
@@
 	(wire
 		(pts
-			(xy 147.32 19.05) (xy 166.37 19.05)
+			(xy 147.32 26.67) (xy 166.37 26.67)
 		)
 		(stroke
@@
 	(wire
 		(pts
-			(xy 208.28 31.75) (xy 208.28 24.13)
+			(xy 208.28 39.37) (xy 208.28 26.67)
 		)
 		(stroke
@@
 	(wire
 		(pts
-			(xy 123.19 19.05) (xy 147.32 19.05)
+			(xy 123.19 26.67) (xy 147.32 26.67)
 		)
 		(stroke
@@
 	(wire
 		(pts
-			(xy 166.37 19.05) (xy 177.8 19.05)
+			(xy 166.37 26.67) (xy 181.61 26.67)
 		)
 		(stroke
@@
 	(wire
 		(pts
-			(xy 185.42 31.75) (xy 185.42 35.56)
+			(xy 185.42 39.37) (xy 185.42 43.18)
 		)
 		(stroke
@@
 	(wire
 		(pts
-			(xy 123.19 16.51) (xy 123.19 19.05)
-		)
-		(stroke
-			(width 0)
-			(type default)
-		)
-	)
-	(wire
-		(pts
 			(xy 119.38 185.42) (xy 123.19 185.42)
 		)
@@
 	(wire
 		(pts
+			(xy 123.19 26.67) (xy 123.19 30.48)
+		)
+		(stroke
+			(width 0)
+			(type default)
+		)
+	)
+	(wire
+		(pts
 			(xy 64.77 129.54) (xy 64.77 139.7)
 		)
@@
 	(wire
 		(pts
-			(xy 208.28 24.13) (xy 207.01 24.13)
+			(xy 208.28 26.67) (xy 207.01 26.67)
 		)
 		(stroke
@@
 	(wire
 		(pts
-			(xy 147.32 31.75) (xy 166.37 31.75)
+			(xy 147.32 39.37) (xy 166.37 39.37)
 		)
 		(stroke
@@
 	(symbol
 		(lib_id "Device:C_Polarized")
-		(at 147.32 25.4 0)
+		(at 147.32 33.02 0)
 		(unit 1)
 		(exclude_from_sim no)
@@
 		(fields_autoplaced yes)
 		(property "Reference" "C6"
-			(at 151.13 23.241 0)
+			(at 151.13 30.861 0)
 			(effects
 				(font
@@
 		)
 		(property "Value" "47uF 16V"
-			(at 151.13 25.781 0)
+			(at 151.13 33.401 0)
 			(effects
 				(font
@@
 		)
 		(property "Footprint" "Capacitor_THT:CP_Radial_D5.0mm_P2.50mm"
-			(at 148.2852 29.21 0)
+			(at 148.2852 36.83 0)
 			(effects
 				(font
@@
 		)
 		(property "Datasheet" "~"
-			(at 147.32 25.4 0)
+			(at 147.32 33.02 0)
 			(effects
 				(font
@@
 		)
 		(property "Description" ""
-			(at 147.32 25.4 0)
+			(at 147.32 33.02 0)
 			(effects
 				(font
@@
 		)
 		(property "Value" "ZTX313"
-			(at 55.626 119.634 0)
+			(at 54.61 119.634 0)
 			(effects
 				(font
@@
 			)
 		)
-		(property "Footprint" "Resistor_THT:R_Axial_DIN0207_L6.3mm_D2.5mm_P10.16mm_Horizontal"
+		(property "Footprint" "Resistor_THT:R_Axial_DIN0207_L6.3mm_D2.5mm_P7.62mm_Horizontal"
 			(at 97.282 167.64 90)
 			(effects
@@
 	(symbol
 		(lib_id "74xx:74HC04")
-		(at 194.31 24.13 90)
+		(at 194.31 26.67 90)
 		(unit 7)
 		(exclude_from_sim no)
@@
 		(dnp no)
 		(property "Reference" "U4"
-			(at 194.564 27.178 90)
+			(at 194.564 29.718 90)
 			(effects
 				(font
@@
 		)
 		(property "Value" "74HC04"
-			(at 194.31 21.336 90)
+			(at 194.31 23.876 90)
 			(effects
 				(font
@@
 		)
 		(property "Footprint" "Package_DIP:DIP-14_W7.62mm"
-			(at 194.31 24.13 0)
+			(at 194.31 26.67 0)
 			(effects
 				(font
@@
 		)
 		(property "Datasheet" "https://assets.nexperia.com/documents/data-sheet/74HC_HCT04.pdf"
-			(at 194.31 24.13 0)
+			(at 194.31 26.67 0)
 			(effects
 				(font
@@
 		)
 		(property "Description" ""
-			(at 194.31 24.13 0)
+			(at 194.31 26.67 0)
 			(effects
 				(font
@@
 	(symbol
 		(lib_id "Device:C")
-		(at 166.37 25.4 0)
+		(at 166.37 33.02 0)
 		(unit 1)
 		(exclude_from_sim no)
@@
 		(dnp no)
 		(property "Reference" "C5"
-			(at 170.18 24.13 0)
+			(at 170.18 31.75 0)
 			(effects
 				(font
@@
 		)
 		(property "Value" "47nF"
-			(at 170.18 26.67 0)
+			(at 170.18 34.29 0)
 			(effects
 				(font
@@
 		)
 		(property "Footprint" "Capacitor_THT:C_Disc_D3.4mm_W2.1mm_P2.50mm"
-			(at 167.3352 29.21 0)
+			(at 167.3352 36.83 0)
 			(effects
 				(font
@@
 		)
 		(property "Datasheet" "~"
-			(at 166.37 25.4 0)
+			(at 166.37 33.02 0)
 			(effects
 				(font
@@
 		)
 		(property "Description" ""
-			(at 166.37 25.4 0)
+			(at 166.37 33.02 0)
 			(effects
 				(font
@@
 			)
 		)
-		(property "Footprint" "Resistor_THT:R_Axial_DIN0207_L6.3mm_D2.5mm_P10.16mm_Horizontal"
+		(property "Footprint" "Capacitor_THT:C_Disc_D3.4mm_W2.1mm_P2.50mm"
 			(at 111.76 186.3852 0)
 			(effects
@@
 	(symbol
 		(lib_id "power:GND")
-		(at 185.42 35.56 0)
+		(at 185.42 43.18 0)
 		(unit 1)
 		(exclude_from_sim no)
@@
 		(fields_autoplaced yes)
 		(property "Reference" "#PWR0104"
-			(at 185.42 41.91 0)
+			(at 185.42 49.53 0)
 			(effects
 				(font
@@
 		)
 		(property "Value" "GND"
-			(at 185.42 40.64 0)
+			(at 185.42 48.26 0)
 			(effects
 				(font
@@
 		)
 		(property "Footprint" ""
-			(at 185.42 35.56 0)
+			(at 185.42 43.18 0)
 			(effects
 				(font
@@
 		)
 		(property "Datasheet" ""
-			(at 185.42 35.56 0)
+			(at 185.42 43.18 0)
 			(effects
 				(font
@@
 		)
 		(property "Description" ""
-			(at 185.42 35.56 0)
+			(at 185.42 43.18 0)
 			(effects
 				(font
@@
 		)
 		(property "Value" "ZTX313"
-			(at 81.534 119.634 0)
+			(at 82.55 119.634 0)
 			(effects
 				(font
@@
 			)
 		)
-		(property "Footprint" "Resistor_THT:R_Axial_DIN0207_L6.3mm_D2.5mm_P10.16mm_Horizontal"
+		(property "Footprint" "Capacitor_THT:C_Disc_D3.4mm_W2.1mm_P2.50mm"
 			(at 95.25 186.3852 0)
 			(effects
